File: hardware/ir-receiver/ir-receiver.kicad_pcb (KiCad board)
At the start: 2 copper layers, 70 x 15 mm, 15 parts, among them IC1 OPA381, X1 Conn_01x04

Commit message: Make receiver PCB two-sided
Parts:
- moved C2 7.11 mm to (149.0, 107.4)
Routing:
- net +5V: track 17.9 -> 5.78 mm
- net GND: track 12.8 -> 20.5 mm, vias 0 -> 13
- net Net-(C1-Pad1): track 18.9 -> 17.0 mm
- added copper zone on F.Cu, net +5V
- added copper zone on B.Cu, net GND
- removed copper zone on F.Cu, net GND

Commit message: Double-sided PCBs
Parts:
- added C3: 100nF, Capacitor_SMD:C_0805_2012Metric_Pad1.15x1.40mm_HandSolder, F.Cu at (207.8, 112.8)
Routing:
- net GND: track 20.5 -> 19.1 mm, vias 13 -> 14
Changed lines of the file:
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@@
     (thickness 1.6)
     (drawings 669)
-    (tracks 65)
-    (modules 15)
+    (tracks 63)
+    (modules 16)
     (nets 6)
   )
   (page "A4")
   (layers
-    (0 "F.Cu" signal)
-    (31 "B.Cu" signal)
+    (0 "F.Cu" signal hide)
+    (31 "B.Cu" signal hide)
     (32 "B.Adhes" user)
     (33 "F.Adhes" user)
@@
     (user_trace_width 0.3)
     (trace_clearance 0.2)
-    (zone_clearance 0.508)
+    (zone_clearance 0.2)
     (zone_45_only no)
     (trace_min 0.15)
@@
     (add_net "Net-(X1-Pad3)")
   )
+  (module "Capacitor_SMD:C_0805_2012Metric_Pad1.15x1.40mm_HandSolder" (layer "F.Cu")
+    (at 207.8 112.8 90)
+    (descr "Capacitor SMD 0805 (2012 Metric), square (rectangular) end terminal, IPC_7351 nominal with elongated pad for handsoldering. (Body size source: https://docs.google.com/spreadsheets/d/1BsfQQcO9C6DZCsRaXUlFlo91Tg2WpOkGARC1WS5S8t0/edit?usp=sharing), generated with kicad-footprint-generator")
+    (tags "capacitor handsolder")
+    (attr smd)
+    (fp_text reference "C3" (at -3 0 180) (layer "F.SilkS")
+      (effects (font (size 1 1) (thickness 0.15)))
+    )
+    (fp_text value "100nF" (at 0 1.65 90) (layer "F.Fab")
+      (effects (font (size 1 1) (thickness 0.15)))
+    )
+    (fp_line (start -1 0.6) (end -1 -0.6) (layer "F.Fab") (width 0.1))
+    (fp_line (start -1 -0.6) (end 1 -0.6) (layer "F.Fab") (width 0.1))
+    (fp_line (start 1 -0.6) (end 1 0.6) (layer "F.Fab") (width 0.1))
+    (fp_line (start 1 0.6) (end -1 0.6) (layer "F.Fab") (width 0.1))
+    (fp_line (start -0.261252 -0.71) (end 0.261252 -0.71) (layer "F.SilkS") (width 0.12))
+    (fp_line (start -0.261252 0.71) (end 0.261252 0.71) (layer "F.SilkS") (width 0.12))
+    (fp_line (start -1.85 0.95) (end -1.85 -0.95) (layer "F.CrtYd") (width 0.05))
+    (fp_line (start -1.85 -0.95) (end 1.85 -0.95) (layer "F.CrtYd") (width 0.05))
+    (fp_line (start 1.85 -0.95) (end 1.85 0.95) (layer "F.CrtYd") (width 0.05))
+    (fp_line (start 1.85 0.95) (end -1.85 0.95) (layer "F.CrtYd") (width 0.05))
+    (fp_text user "%R" (at 0 0 90) (layer "F.Fab")
+      (effects (font (size 0.5 0.5) (thickness 0.08)))
+    )
+    (pad "2" smd roundrect (at 1.025 0 90) (size 1.15 1.4) (layers "F.Cu" "F.Paste" "F.Mask") (roundrect_rratio 0.217391)
+      (net 3 "GND"))
+    (pad "1" smd roundrect (at -1.025 0 90) (size 1.15 1.4) (layers "F.Cu" "F.Paste" "F.Mask") (roundrect_rratio 0.217391)
+      (net 4 "+5V"))
+    (model "${KISYS3DMOD}/Capacitor_SMD.3dshapes/C_0805_2012Metric.wrl"
+      (at (xyz 0 0 0))
+      (scale (xyz 1 1 1))
+      (rotate (xyz 0 0 0))
+    )
+  )
   (module "Connector_PinHeader_2.54mm:PinHeader_1x04_P2.54mm_Vertical" (layer "F.Cu")
     (at 142.6 108.9)
@@
     (tags "SSOP 0.65")
     (attr smd)
-    (fp_text reference "IC1" (at 0 -2.7) (layer "F.SilkS")
+    (fp_text reference "IC1" (at -4.1 -0.1 90) (layer "F.SilkS")
       (effects (font (size 1 1) (thickness 0.15)))
     )
@@
     (effects (font (size 1 1) (thickness 0.15)))
   )
-  (gr_line (start 208 114) (end 207 112) (layer "F.SilkS") (width 0.12))
+  (gr_line (start 154 113.8) (end 153 111.8) (layer "F.SilkS") (width 0.12))
   (gr_text "Infrared Receive Array" (at 181.3 107.6) (layer "F.SilkS")
     (effects (font (size 1.5 1.5) (thickness 0.15)))
   )
-  (gr_line (start 209 112) (end 208 114) (layer "F.SilkS") (width 0.12))
-  (gr_line (start 207 112) (end 209 112) (layer "F.SilkS") (width 0.12))
-  (gr_line (start 207 114) (end 209 114) (layer "F.SilkS") (width 0.12))
-  (gr_line (start 208 111) (end 208 115) (layer "F.SilkS") (width 0.12))
+  (gr_line (start 155 111.8) (end 154 113.8) (layer "F.SilkS") (width 0.12))
+  (gr_line (start 153 111.8) (end 155 111.8) (layer "F.SilkS") (width 0.12))
+  (gr_line (start 153 113.8) (end 155 113.8) (layer "F.SilkS") (width 0.12))
+  (gr_line (start 154 110.8) (end 154 114.8) (layer "F.SilkS") (width 0.12))
   (gr_line (start 140 105) (end 140 120) (layer "Edge.Cuts") (width 0.05))
   (gr_line (start 210 105) (end 140 105) (layer "Edge.Cuts") (width 0.05))
   (gr_line (start 210 120) (end 210 105) (layer "Edge.Cuts") (width 0.05))
   (gr_line (start 140 120) (end 210 120) (layer "Edge.Cuts") (width 0.05))
+  (segment (start 147.3 111.975) (end 148.775 111.975) (width 0.3) (layer "F.Cu") (net 3))
+  (segment (start 148.775 111.975) (end 148.8 112) (width 0.3) (layer "F.Cu") (net 3))
+  (segment (start 207.8 110.3) (end 207.8 111.65) (width 0.3) (layer "F.Cu") (net 3))
+  (via (at 207.8 110.3) (size 0.8) (drill 0.4) (layers "F.Cu" "B.Cu") (net 3))
   (via (at 158 109.2) (size 0.8) (drill 0.4) (layers "F.Cu" "B.Cu") (net 3))
   (segment (start 158 109.2) (end 158 110.55) (width 0.3) (layer "F.Cu") (net 3))
@@
   (segment (start 163 109.4) (end 163 110.75) (width 0.3) (layer "F.Cu") (net 3))
   (via (at 163 109.4) (size 0.8) (drill 0.4) (layers "F.Cu" "B.Cu") (net 3))
-  (via (at 148.9 111.1) (size 0.8) (drill 0.4) (layers "F.Cu" "B.Cu") (net 3))
-  (segment (start 148.9 111.1) (end 148.9 110.9) (width 0.2) (layer "F.Cu") (net 3))
+  (via (at 148.8 112) (size 0.8) (drill 0.4) (layers "F.Cu" "B.Cu") (net 3))
   (segment (start 150.3 114.175) (end 148.3 114.175) (width 0.2) (layer "F.Cu") (net 2))
   (segment (start 150.3 116.225) (end 148.3 116.225) (width 0.2) (layer "F.Cu") (net 1))
@@
   (segment (start 147.3 111.325) (end 146.325 111.325) (width 0.2) (layer "F.Cu") (net 1))
   (segment (start 146.325 111.325) (end 146.1 111.55) (width 0.2) (layer "F.Cu") (net 1))
-  (segment (start 147.3 111.975) (end 148.725 111.975) (width 0.2) (layer "F.Cu") (net 3))
-  (segment (start 148.725 111.975) (end 148.9 111.8) (width 0.2) (layer "F.Cu") (net 3))
-  (segment (start 148.9 111.8) (end 148.9 111.1) (width 0.2) (layer "F.Cu") (net 3))
-  (segment (start 148.675 110.675) (end 147.3 110.675) (width 0.2) (layer "F.Cu") (net 3))
-  (segment (start 148.9 110.9) (end 148.675 110.675) (width 0.2) (layer "F.Cu") (net 3))
   (zone (net 3) (net_name "GND") (layer "B.Cu") (hatch edge 0.508)
     (connect_pads (clearance 0.508))
@@
   )
   (zone (net 4) (net_name "+5V") (layer "F.Cu") (hatch edge 0.508)
-    (connect_pads (clearance 0.508))
-    (min_thickness 0.254)
+    (connect_pads (clearance 0.2))
+    (min_thickness 0.2)
     (fill yes (thermal_gap 0.508) (thermal_bridge_width 0.508))
     (polygon
